File: esp32-c3-02.kicad_sch (KiCad schematic)
At the start: 30 parts, among them J3 GSD090012SEU, U2 USBLC6-2SC6, U3 CP2102N-Axx-xQFN20, U4 W25Q32JVSSIQ, U5 ESP32-C3-WROOM-02-H4

Commit message: ad
Parts:
- C10, C12, C13, C7, C9: footprint (none) -> Capacitor_SMD:C_0805_2012Metric
- C11, C14, C8: footprint (none) -> esp32 footprints:T491A
- LED5, LED6: footprint LEDC2012X120N -> esp32 footprints:LEDC2012X120N
- R11, R12, R13, R14, R15, R16, R17, R18, R19, R20: footprint (none) -> Resistor_SMD:R_0805_2012Metric
- TP1, TP2, TP3, TP4, TP5: footprint (none) -> TestPoint:TestPoint_Pad_D1.0mm
Connections:
- net GND: now also U3.12 (GND), U3.21 (GND), U3.3 (GND)
- no-connect marks 2 -> 7
Changed lines of the file:
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@@
 	)
 	(no_connect
+		(at 95.25 92.71)
+	)
+	(no_connect
+		(at 95.25 77.47)
+	)
+	(no_connect
+		(at 95.25 85.09)
+	)
+	(no_connect
+		(at 95.25 95.25)
+	)
+	(no_connect
+		(at 95.25 87.63)
+	)
+	(no_connect
 		(at 176.53 132.08)
 	)
@@
 	(wire
 		(pts
+			(xy 82.55 113.03) (xy 82.55 114.3)
+		)
+		(stroke
+			(width 0)
+			(type default)
+		)
+	)
+	(wire
+		(pts
 			(xy 148.844 149.098) (xy 153.924 149.098)
 		)
@@
 	)
 	(symbol
+		(lib_id "power:PWR_FLAG")
+		(at 80.01 33.02 270)
+		(unit 1)
+		(exclude_from_sim no)
+		(in_bom yes)
+		(on_board yes)
+		(dnp no)
+		(fields_autoplaced yes)
+		(property "Reference" "#FLG05"
+			(at 81.915 33.02 0)
+			(effects
+				(font
+					(size 1.27 1.27)
+				)
+				(hide yes)
+			)
+		)
+		(property "Value" "PWR_FLAG"
+			(at 83.82 33.0199 90)
+			(effects
+				(font
+					(size 1.27 1.27)
+				)
+				(justify left)
+			)
+		)
+		(property "Footprint" ""
+			(at 80.01 33.02 0)
+			(effects
+				(font
+					(size 1.27 1.27)
+				)
+				(hide yes)
+			)
+		)
+		(property "Datasheet" "~"
+			(at 80.01 33.02 0)
+			(effects
+				(font
+					(size 1.27 1.27)
+				)
+				(hide yes)
+			)
+		)
+		(property "Description" "Special symbol for telling ERC where power comes from"
+			(at 80.01 33.02 0)
+			(effects
+				(font
+					(size 1.27 1.27)
+				)
+				(hide yes)
+			)
+		)
+		(pin "1"
+		)
+		(instances
+			(project "esp32_iot"
+				(path "/0c27022e-f7a1-45ca-b269-a51d4ff975b0/989a141a-e25e-45c3-9987-b10e8b0a6e30"
+					(reference "#FLG05")
+					(unit 1)
+				)
+			)
+		)
+	)
+	(symbol
 		(lib_id "power:GND")
 		(at 59.69 97.79 0)
@@
 			)
 		)
-		(property "Footprint" ""
+		(property "Footprint" "Capacitor_SMD:C_0805_2012Metric"
 			(at 60.96 42.8752 0)
 			(effects
@@
 			)
 		)
-		(property "Footprint" ""
+		(property "Footprint" "esp32 footprints:T491A"
 			(at 272.7452 48.26 0)
 			(effects
@@
 			)
 		)
-		(property "Footprint" ""
+		(property "Footprint" "TestPoint:TestPoint_Pad_D1.0mm"
 			(at 161.29 54.61 0)
 			(effects
@@
 			)
 		)
-		(property "Footprint" ""
+		(property "Footprint" "TestPoint:TestPoint_Pad_D1.0mm"
 			(at 161.29 62.23 0)
 			(effects
@@
 			)
 		)
-		(property "Footprint" ""
+		(property "Footprint" "Resistor_SMD:R_0805_2012Metric"
 			(at 21.082 67.31 90)
 			(effects
@@
 			)
 		)
-		(property "Footprint" ""
+		(property "Footprint" "TestPoint:TestPoint_Pad_D1.0mm"
 			(at 161.29 36.83 0)
 			(effects
@@
 			)
 		)
-		(property "Footprint" ""
+		(property "Footprint" "Resistor_SMD:R_0805_2012Metric"
 			(at 246.38 56.642 90)
 			(effects
@@
 			)
 		)
-		(property "Footprint" ""
+		(property "Footprint" "Resistor_SMD:R_0805_2012Metric"
 			(at 222.25 135.128 90)
 			(effects
@@
 	(symbol
 		(lib_id "power:GND")
+		(at 82.55 114.3 0)
+		(unit 1)
+		(exclude_from_sim no)
+		(in_bom yes)
+		(on_board yes)
+		(dnp no)
+		(fields_autoplaced yes)
+		(property "Reference" "#PWR056"
+			(at 82.55 120.65 0)
+			(effects
+				(font
+					(size 1.27 1.27)
+				)
+				(hide yes)
+			)
+		)
+		(property "Value" "GND"
+			(at 82.55 119.38 0)
+			(effects
+				(font
+					(size 1.27 1.27)
+				)
+				(hide yes)
+			)
+		)
+		(property "Footprint" ""
+			(at 82.55 114.3 0)
+			(effects
+				(font
+					(size 1.27 1.27)
+				)
+				(hide yes)
+			)
+		)
+		(property "Datasheet" ""
+			(at 82.55 114.3 0)
+			(effects
+				(font
+					(size 1.27 1.27)
+				)
+				(hide yes)
+			)
+		)
+		(property "Description" "Power symbol creates a global label with name \"GND\" , ground"
+			(at 82.55 114.3 0)
+			(effects
+				(font
+					(size 1.27 1.27)
+				)
+				(hide yes)
+			)
+		)
+		(pin "1"
+		)
+		(instances
+			(project "esp32_iot"
+				(path "/0c27022e-f7a1-45ca-b269-a51d4ff975b0/989a141a-e25e-45c3-9987-b10e8b0a6e30"
+					(reference "#PWR056")
+					(unit 1)
+				)
+			)
+		)
+	)
+	(symbol
+		(lib_id "power:GND")
 		(at 265.43 57.15 0)
 		(unit 1)
@@
 			)
 		)
-		(property "Footprint" ""
+		(property "Footprint" "Resistor_SMD:R_0805_2012Metric"
 			(at 110.49 89.662 90)
 			(effects
@@
 			)
 		)
-		(property "Footprint" "LEDC2012X120N"
+		(property "Footprint" "esp32 footprints:LEDC2012X120N"
 			(at 134.62 199.06 0)
 			(effects
@@
 			)
 		)
-		(property "Footprint" ""
+		(property "Footprint" "Resistor_SMD:R_0805_2012Metric"
 			(at 43.18 160.528 90)
 			(effects
@@
 			)
 		)
-		(property "Footprint" ""
+		(property "Footprint" "esp32 footprints:T491A"
 			(at 60.96 33.9852 0)
 			(effects
@@
 			)
 		)
-		(property "Footprint" "LEDC2012X120N"
+		(property "Footprint" "esp32 footprints:LEDC2012X120N"
 			(at 134.62 185.09 0)
 			(effects
@@
 			)
 		)
-		(property "Footprint" ""
+		(property "Footprint" "TestPoint:TestPoint_Pad_D1.0mm"
 			(at 161.29 71.12 0)
 			(effects
@@
 			)
 		)
-		(property "Footprint" ""
+		(property "Footprint" "Resistor_SMD:R_0805_2012Metric"
 			(at 21.082 82.55 90)
 			(effects
@@
 			)
 		)
-		(property "Footprint" ""
+		(property "Footprint" "Capacitor_SMD:C_0805_2012Metric"
 			(at 37.7952 86.36 0)
 			(effects
@@
 			)
 		)
-		(property "Footprint" ""
+		(property "Footprint" "Resistor_SMD:R_0805_2012Metric"
 			(at 222.25 126.238 90)
 			(effects
@@
 			)
 		)
-		(property "Footprint" ""
+		(property "Footprint" "Resistor_SMD:R_0805_2012Metric"
 			(at 110.49 103.632 90)
 			(effects
@@
 			)
 		)
-		(property "Footprint" ""
+		(property "Footprint" "Capacitor_SMD:C_0805_2012Metric"
 			(at 97.4852 157.48 0)
 			(effects
@@
 			)
 		)
-		(property "Footprint" ""
+		(property "Footprint" "Resistor_SMD:R_0805_2012Metric"
 			(at 186.69 76.708 90)
 			(effects
@@
 			)
 		)
-		(property "Footprint" ""
+		(property "Footprint" "Capacitor_SMD:C_0805_2012Metric"
 			(at 272.0848 134.62 0)
 			(effects
@@
 			)
 		)
-		(property "Footprint" ""
+		(property "Footprint" "TestPoint:TestPoint_Pad_D1.0mm"
 			(at 161.29 45.72 0)
 			(effects
@@
 			)
 		)
-		(property "Footprint" ""
+		(property "Footprint" "esp32 footprints:T491A"
 			(at 258.1148 134.62 0)
 			(effects
@@
 			)
 		)
-		(property "Footprint" ""
+		(property "Footprint" "Resistor_SMD:R_0805_2012Metric"
 			(at 58.42 64.008 90)
 			(effects
@@
 			)
 		)
-		(property "Footprint" ""
+		(property "Footprint" "Capacitor_SMD:C_0805_2012Metric"
 			(at 258.7752 48.26 0)
 			(effects

Commit message: wip layout 1
Parts:
- J3: footprint GSD090012SEU:AMPHENOL_GSD090012SEU -> esp32 footprints:AMPHENOL_GSD090012SEU
- R19: value 20 -> 50
- U3: footprint Package_DFN_QFN:SiliconLabs_QFN-20-1EP_3x3mm_P0.5mm -> esp32 footprints:QFN50P400X400X100-21N
- U4: footprint W25Q32JVSSIQ:SOIC127P790X216-8N -> esp32 footprints:SOIC127P790X216-8N
- U5: footprint ESP32-C3-WROOM-02-H4:MODULE_ESP32-C3-WROOM-02-H4 -> esp32 footprints:MODULE_ESP32-C3-WROOM-02-H4
Changed lines of the file:
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@@
 	)
 	(junction
-		(at 148.844 171.45)
-		(diameter 0)
-		(color 0 0 0 0)
-	)
-	(junction
 		(at 96.52 146.05)
 		(diameter 0)
@@
 	)
 	(junction
-		(at 148.844 168.91)
-		(diameter 0)
-		(color 0 0 0 0)
-	)
-	(junction
 		(at 80.01 33.02)
 		(diameter 0)
@@
 	)
 	(junction
+		(at 148.844 171.45)
+		(diameter 0)
+		(color 0 0 0 0)
+	)
+	(junction
 		(at 148.844 179.07)
 		(diameter 0)
@@
 	)
 	(junction
+		(at 148.844 168.91)
+		(diameter 0)
+		(color 0 0 0 0)
+	)
+	(junction
 		(at 36.83 74.93)
 		(diameter 0)
@@
 	(wire
 		(pts
+			(xy 148.844 168.91) (xy 152.4 168.91)
+		)
+		(stroke
+			(width 0)
+			(type default)
+		)
+	)
+	(wire
+		(pts
 			(xy 68.58 33.02) (xy 80.01 33.02)
 		)
@@
 	(wire
 		(pts
-			(xy 148.59 179.07) (xy 148.844 179.07)
+			(xy 148.59 168.91) (xy 148.844 168.91)
 		)
 		(stroke
@@
 	(wire
 		(pts
-			(xy 148.59 181.61) (xy 148.844 181.61)
+			(xy 148.59 179.07) (xy 148.844 179.07)
 		)
 		(stroke
@@
 	(wire
 		(pts
-			(xy 246.38 34.29) (xy 246.38 36.83)
+			(xy 148.59 181.61) (xy 148.844 181.61)
 		)
 		(stroke
@@
 	(wire
 		(pts
-			(xy 148.844 171.45) (xy 152.4 171.45)
+			(xy 246.38 34.29) (xy 246.38 36.83)
 		)
 		(stroke
@@
 	(wire
 		(pts
+			(xy 148.844 171.45) (xy 152.4 171.45)
+		)
+		(stroke
+			(width 0)
+			(type default)
+		)
+	)
+	(wire
+		(pts
 			(xy 35.56 158.75) (xy 39.37 158.75)
 		)
@@
 	(wire
 		(pts
-			(xy 148.844 168.91) (xy 152.4 168.91)
-		)
-		(stroke
-			(width 0)
-			(type default)
-		)
-	)
-	(wire
-		(pts
 			(xy 118.11 168.91) (xy 123.19 168.91)
 		)
@@
 	(wire
 		(pts
+			(xy 148.59 171.45) (xy 148.844 171.45)
+		)
+		(stroke
+			(width 0)
+			(type default)
+		)
+	)
+	(wire
+		(pts
 			(xy 218.44 132.08) (xy 218.44 133.35)
 		)
@@
 	(wire
 		(pts
-			(xy 148.59 168.91) (xy 148.844 168.91)
-		)
-		(stroke
-			(width 0)
-			(type default)
-		)
-	)
-	(wire
-		(pts
-			(xy 148.59 171.45) (xy 148.844 171.45)
-		)
-		(stroke
-			(width 0)
-			(type default)
-		)
-	)
-	(wire
-		(pts
 			(xy 226.06 124.46) (xy 231.14 124.46)
 		)
@@
 			)
 		)
-		(property "Footprint" "W25Q32JVSSIQ:SOIC127P790X216-8N"
+		(property "Footprint" "esp32 footprints:SOIC127P790X216-8N"
 			(at 73.66 153.67 0)
 			(effects
@@
 			)
 		)
-		(property "Footprint" "Package_DFN_QFN:SiliconLabs_QFN-20-1EP_3x3mm_P0.5mm"
+		(property "Footprint" "esp32 footprints:QFN50P400X400X100-21N"
 			(at 114.3 111.76 0)
 			(effects
@@
 			)
 		)
-		(property "Value" "20"
+		(property "Value" "50"
 			(at 186.69 71.12 90)
 			(effects
@@
 			)
 		)
-		(property "Footprint" "ESP32-C3-WROOM-02-H4:MODULE_ESP32-C3-WROOM-02-H4"
+		(property "Footprint" "esp32 footprints:MODULE_ESP32-C3-WROOM-02-H4"
 			(at 220.98 69.85 0)
 			(effects
@@
 			)
 		)
-		(property "Footprint" "GSD090012SEU:AMPHENOL_GSD090012SEU"
+		(property "Footprint" "esp32 footprints:AMPHENOL_GSD090012SEU"
 			(at 194.31 132.08 0)
 			(effects
