File: esp32_iot.kicad_sch (KiCad schematic)
At the start: 25 parts, among them J1 B2B-PH-SM4-TB, J2 SS-52400-002, U1 MCP73871

Commit message: ad
Parts:
- C1, C2, C3, C6: footprint (none) -> Capacitor_SMD:C_0805_2012Metric
- C4, C5: footprint (none) -> esp32 footprints:T491A
- F1: footprint FUSC3226X100N -> esp32 footprints:FUSC3226X100N
- LED1, LED2, LED3, LED4: footprint LEDC2012X120N -> esp32 footprints:LEDC2012X120N
- R1, R10, R2, R3, R4, R5, R6, R7, R8, R9: footprint (none) -> Resistor_SMD:R_0805_2012Metric
Connections:
- net GND: now also U1.3 (SEL)

Commit message: wip layout 1
Parts:
- J1: footprint B2B-PH-SM4-TB:JST_B2B-PH-SM4-TB -> esp32 footprints:JST_B2B-PH-SM4-TB
- J2: footprint SS-52400-002:BELFUSE_SS-52400-002 -> esp32 footprints:BELFUSE_SS-52400-002
- VR1: footprint LM1117MPX-3.3:VREG_LM1117MPX-3.3 -> esp32 footprints:VREG_LM1117MPX-3.3
Changed lines of the file:
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@@
 			)
 		)
-		(property "Footprint" "SS-52400-002:BELFUSE_SS-52400-002"
+		(property "Footprint" "esp32 footprints:BELFUSE_SS-52400-002"
 			(at 68.58 71.12 0)
 			(effects
@@
 			)
 		)
-		(property "Footprint" "B2B-PH-SM4-TB:JST_B2B-PH-SM4-TB"
+		(property "Footprint" "esp32 footprints:JST_B2B-PH-SM4-TB"
 			(at 40.64 175.26 0)
 			(effects
@@
 			)
 		)
-		(property "Footprint" "LM1117MPX-3.3:VREG_LM1117MPX-3.3"
+		(property "Footprint" "esp32 footprints:VREG_LM1117MPX-3.3"
 			(at 68.58 129.54 0)
 			(effects
