File: interface.kicad_sch (KiCad schematic)
At the start: 11 parts, among them Q1 BC817

Commit message: ad
Parts:
- C16: footprint (none) -> Capacitor_SMD:C_0805_2012Metric
- C20: renamed from C?; footprint (none) -> Capacitor_SMD:C_0805_2012Metric
- J4: renamed from J?; footprint (none) -> Connector_PinHeader_2.54mm:PinHeader_1x04_P2.54mm_Vertical
- J5: renamed from J?; footprint (none) -> Connector_PinHeader_2.54mm:PinHeader_1x05_P2.54mm_Vertical
- R26: footprint (none) -> Resistor_SMD:R_0805_2012Metric
- R31, R32: renamed from R?; footprint (none) -> Resistor_SMD:R_0805_2012Metric
- gave numbers to parts that had none: 2
Changed lines of the file:
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@@
 		(on_board yes)
 		(dnp no)
-		(property "Reference" "S?"
+		(property "Reference" "S2"
 			(at 164.846 50.8 0)
 			(effects
@@
 			(project ""
 				(path "/0c27022e-f7a1-45ca-b269-a51d4ff975b0/989a141a-e25e-45c3-9987-b10e8b0a6e30/da21be88-f029-4562-8bcb-7645a8dde34c"
-					(reference "S?")
+					(reference "S2")
 					(unit 1)
 				)
@@
 		(on_board yes)
 		(dnp no)
-		(property "Reference" "J?"
+		(property "Reference" "J5"
 			(at 93.98 115.5701 0)
 			(effects
@@
 			)
 		)
-		(property "Footprint" ""
+		(property "Footprint" "Connector_PinHeader_2.54mm:PinHeader_1x05_P2.54mm_Vertical"
 			(at 92.71 114.3 0)
 			(effects
@@
 			(project ""
 				(path "/0c27022e-f7a1-45ca-b269-a51d4ff975b0/989a141a-e25e-45c3-9987-b10e8b0a6e30/da21be88-f029-4562-8bcb-7645a8dde34c"
-					(reference "J?")
+					(reference "J5")
 					(unit 1)
 				)
@@
 			)
 		)
-		(property "Footprint" ""
+		(property "Footprint" "Resistor_SMD:R_0805_2012Metric"
 			(at 157.48 133.858 90)
 			(effects
@@
 		(dnp no)
 		(fields_autoplaced yes)
-		(property "Reference" "R?"
+		(property "Reference" "R31"
 			(at 157.48 105.41 90)
 			(effects
@@
 			)
 		)
-		(property "Footprint" ""
+		(property "Footprint" "Resistor_SMD:R_0805_2012Metric"
 			(at 157.48 113.538 90)
 			(effects
@@
 			(project ""
 				(path "/0c27022e-f7a1-45ca-b269-a51d4ff975b0/989a141a-e25e-45c3-9987-b10e8b0a6e30/da21be88-f029-4562-8bcb-7645a8dde34c"
-					(reference "R?")
+					(reference "R31")
 					(unit 1)
 				)
@@
 		(dnp no)
 		(fields_autoplaced yes)
-		(property "Reference" "C?"
+		(property "Reference" "C20"
 			(at 156.21 77.4699 0)
 			(effects
@@
 			)
 		)
-		(property "Footprint" ""
+		(property "Footprint" "Capacitor_SMD:C_0805_2012Metric"
 			(at 153.3652 82.55 0)
 			(effects
@@
 			(project ""
 				(path "/0c27022e-f7a1-45ca-b269-a51d4ff975b0/989a141a-e25e-45c3-9987-b10e8b0a6e30/da21be88-f029-4562-8bcb-7645a8dde34c"
-					(reference "C?")
+					(reference "C20")
 					(unit 1)
 				)
@@
 		(dnp no)
 		(fields_autoplaced yes)
-		(property "Reference" "Q?"
+		(property "Reference" "Q3"
 			(at 184.15 110.4899 0)
 			(effects
@@
 			(project ""
 				(path "/0c27022e-f7a1-45ca-b269-a51d4ff975b0/989a141a-e25e-45c3-9987-b10e8b0a6e30/da21be88-f029-4562-8bcb-7645a8dde34c"
-					(reference "Q?")
+					(reference "Q3")
 					(unit 1)
 				)
@@
 		(dnp no)
 		(fields_autoplaced yes)
-		(property "Reference" "R?"
+		(property "Reference" "R32"
 			(at 199.39 59.6899 0)
 			(effects
@@
 			)
 		)
-		(property "Footprint" ""
+		(property "Footprint" "Resistor_SMD:R_0805_2012Metric"
 			(at 195.072 60.96 90)
 			(effects
@@
 			(project ""
 				(path "/0c27022e-f7a1-45ca-b269-a51d4ff975b0/989a141a-e25e-45c3-9987-b10e8b0a6e30/da21be88-f029-4562-8bcb-7645a8dde34c"
-					(reference "R?")
+					(reference "R32")
 					(unit 1)
 				)
@@
 		(on_board yes)
 		(dnp no)
-		(property "Reference" "J?"
+		(property "Reference" "J4"
 			(at 91.44 74.9301 0)
 			(effects
@@
 			)
 		)
-		(property "Footprint" ""
+		(property "Footprint" "Connector_PinHeader_2.54mm:PinHeader_1x04_P2.54mm_Vertical"
 			(at 90.17 72.39 0)
 			(effects
@@
 			(project ""
 				(path "/0c27022e-f7a1-45ca-b269-a51d4ff975b0/989a141a-e25e-45c3-9987-b10e8b0a6e30/da21be88-f029-4562-8bcb-7645a8dde34c"
-					(reference "J?")
+					(reference "J4")
 					(unit 1)
 				)
@@
 			)
 		)
-		(property "Footprint" ""
+		(property "Footprint" "Capacitor_SMD:C_0805_2012Metric"
 			(at 204.1652 82.55 0)
 			(effects

Commit message: wip layout 1
Parts:
- S1, S2: footprint USLPT2819DT2TR:SW_USLPT2819DT2TR -> esp32 footprints:SW_USLPT2819DT2TR
Changed lines of the file:
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@@
 			"AAAAAAAAAAAAAAAAAKQgAAAAAAAAAAAAAAAAAAA3BwAAAAAAALERAAAAAAAAJSIAAAAAAAChKQAA"
 			"AAAAAAAAAAAAAAAAAAAAAAAAAAAAAAAAAAAAAAAAAAAAAAAAwgIAAAAAAACqJgAAAAAAAD0NAAAA"
-			"AAAAAAAAAAAAAAAAAAAAAAAAAD4QAAAAAAAAOBkAAAAAAA=="
+			"AAAAAAAAAAAAAAAAAAAAAAAAAD4QAAAAAAAAOBkAAAAAAAAKAAAAIAAAAFMAAABvAAAAIAAAAGgA"
+			"AABlAAAAcgAAAGUAAAAnAAAAcwAAACAAAABoAAAAbwAAAHcAAAAgAAAAaQAAAHQAAAAgAAAAdwAA"
+			"AG8AAAByAAAAawAAAHMAAAA6AAAAIAAAAG8AAABuAAAAYwAAAGUAAAAgAAAAeQAAAG8AAAB1AAAA"
+			"IAAAAGgAAABhAAAAdgAAAGUAAAAgAAAAYwAAAG8AAABtAAAAcAAAAGwAAABlAAAAdAAAAGUAAABk"
+			"AAAAIAAAAHQAAABoAAAAZQAAACAAAABsAAAAYQAAAHkAAABvAAAAdQAAAHQAAAAsAAAAIAAAAGEA"
+			"AABsAAAAbAAAACAAAAB5AAAAbwAAAHUAAAAgAAAAbgAAAGUAAABlAAAAZAAAACAAAAB0AAAAbwAA"
+			"ACAAAABkAAAAbwAAACAAAABpAAAAcwAAACAAAABnAAAAbwAAACAAAAB0AAAAbwAAACAAAABUAAAA"
+			"bwAAAG8AAABsAAAAcwAAACAAAABhAAAAbgAAAGQAAAAgAAAARQAAAHgAAAB0AAAAZQAAAHIAAABu"
+			"AAAAYQAAAGwAAAAgAAAAUAAAAGwAAAB1AAAAZwAAAGkAAABuAAAAcwAAACwAAAAgAAAAYQAAAG4A"
+			"AABkAAAAIAAAAHMAAABlAAAAbAAAAGUAAABjAAAAdAAAACAAAABTAAAAaQAAAGUAAAByAAAAcgAA"
+			"AGEAAAAgAAAAQwAAAGkAAAByAAAAYwAAAHUAAABpAAAAdAAAAHMAAAAgAAAAUQAAAHUAAABvAAAA"
+			"dAAAAGUAAAAuAAAACgAAACAAAABBAAAAIAAAAHcAAABpAAAAbgAAAGQAAABvAAAAdwAAACAAAAB3"
+			"AAAAaQAAAGwAAABsAAAAIAAAAHAAAABvAAAAcAAAAC0AAAB1AAAAcAAAACAAAABhAAAAbgAAAGQA"
+			"AAAgAAAAcwAAAGgAAABvAAAAdwAAACAAAAB0AAAAaAAAAGUAAAAgAAAAcwAAAHAAAABlAAAAYwAA"
+			"AGkAAABmAAAAaQAAAGMAAABhAAAAdAAAAGkAAABvAAAAbgAAAHMAAAAuAAAAIAAAAE8AAAB1AAAA"
+			"cgAAACAAAABwAAAAbAAAAHUAAABnAAAAaQAAAG4AAAAgAAAAcgAAAGUAAABhAAAAZAAAAHMAAAAg"
+			"AAAAdAAAAGgAAABlAAAAIAAAAGQAAABlAAAAcwAAAGkAAABnAAAAbgAAACAAAABmAAAAbwAAAHIA"
+			"AAAgAAAAYQAAACAAAABzAAAAbQAAAG8AAABvAAAAdAAAAGgAAAAgAAAAcQAAAHUAAABvAAAAdAAA"
+			"AGUAAAAgAAAAcAAAAHIAAABvAAAAYwAAAGUAAABzAAAAcw=="
 		)
 	)
@@
 			)
 		)
-		(property "Footprint" "USLPT2819DT2TR:SW_USLPT2819DT2TR"
+		(property "Footprint" "esp32 footprints:SW_USLPT2819DT2TR"
 			(at 165.1 66.04 0)
 			(effects
@@
 			)
 		)
-		(property "Footprint" "USLPT2819DT2TR:SW_USLPT2819DT2TR"
+		(property "Footprint" "esp32 footprints:SW_USLPT2819DT2TR"
 			(at 215.9 66.04 0)
 			(effects
